Commit message: hi

File: src/traktor/urdf/car.urdf (robot description, URDF)
Before this commit: robot moveon, 6 links, 5 joints
Links:
- removed link left_rear_steering_link
- removed link left_rear_wheel
- removed link sag_dif
- removed link sag_on
- added link gps_link, mass 0.1
- added link sag_arka, mass 10; collision cylinder length=0.3 radius=0.4; visual cylinder length=0.20 radius=0.4
- added link sag_arka_dif; visual cylinder length=0.05 radius=0.02
- added link sag_on_dif; visual cylinder length=0.05 radius=0.02
- added link sag_on_teker, mass 10; collision cylinder length=0.3 radius=0.25; visual cylinder length=0.20 radius=0.25
- added link sol_arka, mass 10; collision cylinder length=0.3 radius=0.4; visual cylinder length=0.20 radius=0.4
- added link sol_arka_dif; visual cylinder length=0.05 radius=0.02
- added link sol_on, mass 10; collision cylinder length=0.3 radius=0.25; visual cylinder length=0.20 radius=0.25
- added link sol_on_dif; visual cylinder length=0.05 radius=0.02
Joints:
- removed joint l_r_w_j
- removed joint left_rear_steering_joint
- removed joint sag_dif_joint
- removed joint sag_dif_sag_teker
- added joint gps_joint: type fixed, parent base_link, child gps_link, origin xyz=0 0 1 rpy=0 0 0
- added joint sag_arka_dif_joint: type revolute, parent base_link, child sag_arka_dif, origin xyz=-1.25 -0.85 -0.5 rpy=1.5707 0 0, axis 0 1 0, limit lower=-1 upper=1 effort=100 velocity=1
- added joint sag_arka_dif_sag_arka_teker: type continuous, parent sag_arka_dif, child sag_arka, origin xyz=0.0 0.0 0.0 rpy=0 0 0, axis 0 0 -1, limit effort=100 velocity=100
- added joint sag_on_dif_joint: type revolute, parent base_link, child sag_on_dif, origin xyz=0.75 -0.85 -0.5 rpy=1.5707 0 0, axis 0 1 0, limit lower=-1 upper=1 effort=100 velocity=1
- added joint sag_on_dif_sag_on_teker: type continuous, parent sag_on_dif, child sag_on_teker, origin xyz=0.0 0.0 0.0 rpy=0 0 0, axis 0 0 -1, limit effort=100 velocity=100
- added joint sol_arka_dif_joint: type revolute, parent base_link, child sol_arka_dif, origin xyz=-1.25 0.85 -0.5 rpy=1.5707 0 0, axis 0 1 0, limit lower=-1 upper=1 effort=100 velocity=1
- added joint sol_arka_dif_sol_arka_teker: type continuous, parent sol_arka_dif, child sol_arka, origin xyz=0.0 0.0 0.0 rpy=0 0 0, axis 0 0 -1, limit effort=100 velocity=100
- added joint sol_on_dif_joint: type revolute, parent base_link, child sol_on_dif, origin xyz=0.75 0.85 -0.5 rpy=1.5707 0 0, axis 0 1 0, limit lower=-1 upper=1 effort=100 velocity=1
- added joint sol_on_dif_sol_on_teker: type continuous, parent sol_on_dif, child sol_on, origin xyz=0.0 0.0 0.0 rpy=0 0 0, axis 0 0 -1, limit effort=100 velocity=100

Commit message: traktor urdf changed car.urdf

File: src/traktor/urdf/car.urdf (robot description, URDF)
Before this commit: robot moveon, 11 links, 10 joints
Links:
- removed link gps_link
- removed link sag_arka_dif
- removed link sol_arka_dif
- added link direksiyon, mass 1; collision cylinder length=0.05 radius=0.2; visual cylinder length=0.05 radius=0.2
Joints:
- removed joint gps_joint
- removed joint sag_arka_dif_sag_arka_teker
- removed joint sol_arka_dif_sol_arka_teker
- added joint direksiyon_joint: type revolute, parent base_link, child direksiyon, origin xyz=0.25 0 1 rpy=0 -1 0, axis 0 0 1, limit lower=-1 upper=1 effort=100 velocity=1
- joint sag_arka_dif_joint: axis 0 1 0 -> 0 0 1; child sag_arka_dif -> sag_arka; limit lower=-1 upper=1 effort=100 velocity=1 -> effort=100 velocity=100; origin xyz=-1.25 -0.85 -0.5 rpy=1.5707 0 0 -> xyz=-1.25 -0.85 -0.35 rpy=1.5707 0 0; type revolute -> continuous
- joint sol_arka_dif_joint: axis 0 1 0 -> 0 0 -1; child sol_arka_dif -> sol_arka; limit lower=-1 upper=1 effort=100 velocity=1 -> effort=100 velocity=100; origin xyz=-1.25 0.85 -0.5 rpy=1.5707 0 0 -> xyz=-1.25 0.85 -0.35 rpy=1.5707 0 0; type revolute -> continuous
